File: CMRI-Bus-Interface.sch (EAGLE design)
At the start: 16 parts, among them U1 MAX3465CPD

Commit message: TXEN and RX were shorted
Parts:
- removed RS485IN1: CMRInet Hdr Rt, SPCoast:CONNECTOR-CMRINET.156
- removed RS485IN2: CMRInet Hdr Top, SPCoast:CONNECTOR-CMRINET.156
- added CMRINET3, CMRINET4: CMRInet, SPCoast:CONNECTOR-CMRINET.156
- CMRINET1, CMRINET2: value (none) -> CMRInet
- renumbered CMRINETTOP to CMRINET2, CMRINETTOP1 to CMRINET1
Connections:
- removed net N$36: CMRINET1.4, CMRINET2.4, RS485IN1.4, RS485IN2.4, U1.A
- removed net N$56: CMRINET1.3, CMRINET2.3, RS485IN1.3, RS485IN2.3, U1.B
- removed net N$59: CMRINET1.2, CMRINET2.2, RS485IN1.2, RS485IN2.2, U1.Y
- removed net N$60: CMRINET1.1, CMRINET2.1, RS485IN1.1, RS485IN2.1, U1.Z
- new net IN+: CMRINET1.4, CMRINET2.4, CMRINET3.4, CMRINET4.4, U1.A
- new net IN-: CMRINET1.3, CMRINET2.3, CMRINET3.3, CMRINET4.3, U1.B
- new net OUT+: CMRINET1.2, CMRINET2.2, CMRINET3.2, CMRINET4.2, U1.Y
- new net OUT-: CMRINET1.1, CMRINET2.1, CMRINET3.1, CMRINET4.1, U1.Z
- net SHIELD: now also CMRINET3.5, CMRINET4.5; no longer RS485IN1.5, RS485IN2.5
